File: version_2/hardware/pcb/rev_1/mainboard_v2_r1/schematics/GNSS.kicad_sch (KiCad schematic)
At the start: 2 parts, among them J15 Conn_01x08

Commit message: Small uncertain KiCad update to the files
Other:
- note added: "Ajouter timepulse prochaine révision"
Changed lines of the file:
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@@
 	(generator_version "10.0")
 	(paper "A4")
+	(text "Ajouter timepulse prochaine révision"
+		(exclude_from_sim no)
+		(at 153.924 91.694 0)
+		(effects
+			(font
+				(size 1.27 1.27)
+				(color 255 0 255 1)
+			)
+		)
+	)
 	(junction
 		(at 138.43 113.03)
@@
 			)
 		)
-		(property "Sim.Enable" ""
-			(at 128.27 107.95 0)
-			(hide yes)
-			(show_name no)
-			(do_not_autoplace no)
-			(effects
-				(font
-					(size 1.27 1.27)
-				)
-			)
-		)
 		(pin "2"
 		)
@@
 			(at 138.43 116.84 0)
 			(hide yes)
-			(show_name no)
-			(do_not_autoplace no)
-			(effects
-				(font
-					(size 1.27 1.27)
-				)
-			)
-		)
-		(property "Sim.Enable" ""
-			(at 138.43 116.84 0)
-			(hide yes)
