File: version_2/hardware/pcb/rev_1/simulation/magnetic_board_v2_r1_simu/magnetic_board_v2_r1_simu.kicad_sch (KiCad schematic)
At the start: 25 parts, among them U1 HMC1001_SPICE, U2 INA851_Spice, U3 ${SIM.PARAMS}, U4 ${SIM.PARAMS}

Commit message: Add magnetic board simulation models and improve recording tools
Add tested SPICE models and a Helmholtz simulation workbook, with updated lab notes. Rename the shared Python decoder package to geophys-recording and extend the recording viewer with nominal thermistor temperature, channel defaults, and portable launch paths.
Parts:
- removed V5: 0, symbol Simulation_SPICE:VDC
- added C16: 4u7, Capacitor_THT:C_Rect_L18.0mm_W7.0mm_P15.00mm_FKS3_FKP3, symbol Device:C
- added L1: HELMHOLTZ_PAIR, symbol simulation:helmholtz_coil
- added R6: 100, symbol Device:R
- C14: value 10u -> 4u7
- V1: value 9 -> 5.67
Connections:
- net 0: no longer V3.2
- net FIELD: now also L1.3 (FIELD); no longer V3.1
- net Vint+: now also C16.2
- net at C14.1, R10.2, R14.1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: now also C16.1
- net +4V5 renamed Vb/2
- net +9Vb renamed Vb
- new net: L1.1 (IN), R6.2
- new net: L1.2 (RETURN), V3.2
- new net: R6.1, V3.1
Other:
- note added: ".param FREQ=10"
- note added: "SIN(0 2.5 {FREQ})"
- note removed: ".param A=10m"
- moved on the sheet: C1, C14, C15, C28, MES1, R1, R10, R11, R12, R13, R14, R15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
